Commit message: still figuring out how to rotate in place

File: models/bob.urdf (robot description, URDF)
Before this commit: robot bob, 4 links, 3 joints
Links:
- link base: geometry visual box size=0.3 0.6 0.3
- link rack: geometry visual box size=0.05 0.5 0.05
Joints:
- joint rack_to_left_fork: origin xyz=0.25 -0.15 0.025 rpy=0 0 0 -> xyz=0.25 -0.25 0.025 rpy=0 0 0
- joint rack_to_right_fork: origin xyz=0.25 0.15 0.025 rpy=0 0 0 -> xyz=0.25 0.25 0.025 rpy=0 0 0
